File: xmos.kicad_sch (KiCad schematic)
At the start: 80 parts, among them J4 XMOS JTAG, Q1 LBSS138WT1G, Q2 LBSS138WT1G, Q3 BC847B, U10 XU316-1024-QF60B-C24, U11 W25Q32JVSSIQ, U12 SN74LVC125APWR, U13 TLV73333PDBVR, U16 TS3USB221ERSER, X1 24MHz 12pF

Commit message: rev A2 (rotations corrected after the JLCPCB preview) — 2026-10-02, from rev-a2-endstand (f736024)
Parts:
- R35: LCSC Part # C25130 -> C100510; MPN 0402WGF6800TCE -> CR0402FF6800G; Manufacturer UNI-ROYAL(Uniroyal Elec) -> LIZ Elec; Manufacturer Part 0402WGF6800TCE -> CR0402FF6800G; Power Rating 5% -> 62.5mW; SKU 301010505 -> (none); Status Combox Pro -> (none); Temperature -55°C to 155°C -> -55°C to 125°C
Changed lines of the file:
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@@
 			)
 		)
-		(property "Description" "SMD RES 680R-5%-1/16W;0402"
+		(property "Description" "SMD RES 680R-1%-1/16W;0402"
 			(at 102.87 154.94 0)
 			(effects
@@
 			)
 		)
-		(property "Manufacturer" "UNI-ROYAL(Uniroyal Elec)"
+		(property "Manufacturer" "LIZ Elec"
 			(at 102.87 154.94 0)
 			(effects
@@
 			)
 		)
-		(property "MPN" "0402WGF6800TCE"
+		(property "MPN" "CR0402FF6800G"
 			(at 102.87 154.94 0)
 			(effects
@@
 			)
 		)
-		(property "SKU" "301010505"
+		(property "SKU" ""
 			(at 102.87 154.94 0)
 			(effects
@@
 			)
 		)
-		(property "Power Rating" "5%"
+		(property "Power Rating" "62.5mW"
 			(at 104.775 157.48 90)
 			(effects
@@
 			)
 		)
-		(property "Status" "Combox Pro"
+		(property "Status" ""
 			(at 102.87 154.94 0)
 			(effects
@@
 			)
 		)
-		(property "Temperature" "-55°C to 155°C"
+		(property "Temperature" "-55°C to 125°C"
 			(at 102.87 154.94 0)
 			(effects
@@
 			)
 		)
-		(property "LCSC Part #" "C25130"
+		(property "LCSC Part #" "C100510"
 			(at 102.87 154.94 90)
 			(effects
@@
 			)
 		)
-		(property "Manufacturer Part" "0402WGF6800TCE"
+		(property "Manufacturer Part" "CR0402FF6800G"
 			(at 102.87 154.94 90)
 			(effects
